File: KiCad/Esquema_Mod_Buzzer/Esquema_Buzzer.kicad_sch (KiCad schematic)
At the start: 7 parts, among them J1 XT30-M, M1 Motor_Servo, Q1 BC337, U1 817B, U2 MT3608

Commit message: [ADD] Projetos KiCAD
Parts:
- added C1, C2: C, symbol Device:C
- added R2, R3: R, symbol Device:R
- added U3: MT3608, Package_TO_SOT_SMD:SOT-23-6, symbol Regulator_Switching:MT3608
