File: KiCad/Esquema_Mod_Buzzer/Esquema_Buzzer.kicad_pcb (KiCad board)
At the start: 2 copper layers, 0 parts

Commit message: [ADD] atualizacoes modulos SD
Routing:
- removed copper zone on F.Cu, net (none)
Changed lines of the file:
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@@
 			(outputformat 1)
 			(mirror no)
-			(drillshape 1)
+			(drillshape 0)
 			(scaleselection 1)
-			(outputdirectory "")
+			(outputdirectory "./")
 		)
 	)
@@
 	(gr_text "U1"
 		(at 36 34 0)
-		(layer "F.Cu")
+		(layer "F.SilkS")
 		(effects
 			(font
@@
 	(gr_text "C"
 		(at 39 33 0)
-		(layer "F.Cu")
+		(layer "F.SilkS")
 		(effects
 			(font
@@
 	(gr_text "M1"
 		(at 29.5 34 0)
-		(layer "F.Cu")
+		(layer "F.SilkS")
 		(effects
 			(font
@@
 	(gr_text "R1 + BZ1"
 		(at 36 30 0)
-		(layer "F.Cu")
+		(layer "F.SilkS")
 		(effects
 			(font
@@
 	(gr_text "C"
 		(at 42.5 33.5 0)
-		(layer "F.Cu")
+		(layer "F.SilkS")
 		(effects
 			(font
@@
 	(gr_text "U2-"
 		(at 39.5 38.5 0)
-		(layer "F.Cu")
+		(layer "F.SilkS")
 		(effects
 			(font
@@
 	(gr_text "E"
 		(at 42.5 37 0)
-		(layer "F.Cu")
+		(layer "F.SilkS")
 		(effects
 			(font
@@
 	(gr_text "Q1"
 		(at 42 34.5 0)
-		(layer "F.Cu")
+		(layer "F.SilkS")
 		(effects
 			(font
@@
 	(gr_text "Anode"
 		(at 33 33 0)
-		(layer "F.Cu")
+		(layer "F.SilkS")
 		(effects
 			(font
@@
 	(gr_text "E"
 		(at 39 35 0)
-		(layer "F.Cu")
+		(layer "F.SilkS")
 		(effects
 			(font
@@
 	(gr_text "+"
 		(at 33 30 0)
-		(layer "F.Cu")
+		(layer "F.SilkS")
 		(effects
 			(font
@@
 	(gr_text "B"
 		(at 43 35 0)
-		(layer "F.Cu")
+		(layer "F.SilkS")
 		(effects
 			(font
@@
 	(gr_text "Cathode"
 		(at 33 35 0)
-		(layer "F.Cu")
+		(layer "F.SilkS")
 		(effects
 			(font
@@
 	(gr_text "-"
 		(at 41.5 30 0)
-		(layer "F.Cu")
+		(layer "F.SilkS")
 		(effects
 			(font
@@
 	(gr_text "J1+"
 		(at 37 38.5 0)
-		(layer "F.Cu")
+		(layer "F.SilkS")
 		(effects
 			(font
@@
 	(gr_text "U2+"
 		(at 29.5 29.5 0)
-		(layer "F.Cu")
+		(layer "F.SilkS")
 		(effects
 			(font
@@
 		(net 0)
 		(net_name "")
-		(layer "F.Cu")
-		(name "J1")
+		(layers "F.Cu" "F.SilkS")
+		(name "Resistor 1k")
 		(hatch edge 0.5)
 		(connect_pads
@@
 		(polygon
 			(pts
-				(xy 36.5 38.5) (xy 36.5 36.5) (xy 38.5 36.5) (xy 38.5 38.5)
-			)
-		)
-	)
-	(zone
-		(net 0)
-		(net_name "")
-		(layer "F.Cu")
-		(name "Resistor 1k")
+				(xy 43 31) (xy 32 31) (xy 32 29) (xy 43 29)
+			)
+		)
+	)
+	(zone
+		(net 0)
+		(net_name "")
+		(layers "F.Cu" "F.SilkS")
+		(name "U2")
 		(hatch edge 0.5)
 		(connect_pads
@@
 		(polygon
 			(pts
-				(xy 43 31) (xy 32 31) (xy 32 29) (xy 43 29)
-			)
-		)
-	)
-	(zone
-		(net 0)
-		(net_name "")
-		(layer "F.Cu")
-		(name "U2")
+				(xy 41 38.5) (xy 39 38.5) (xy 39 36.5) (xy 41 36.5)
+			)
+		)
+	)
+	(zone
+		(net 0)
+		(net_name "")
+		(layers "F.Cu" "F.SilkS")
+		(name "M1")
 		(hatch edge 0.5)
 		(connect_pads
@@
 		(polygon
 			(pts
-				(xy 41 38.5) (xy 39 38.5) (xy 39 36.5) (xy 41 36.5)
-			)
-		)
-	)
-	(zone
-		(net 0)
-		(net_name "")
-		(layer "F.Cu")
-		(name "transistor")
+				(xy 29 31.5) (xy 31 31.5) (xy 31 36) (xy 29 36)
+			)
+		)
+	)
+	(zone
+		(net 0)
+		(net_name "")
+		(layer "F.SilkS")
+		(name "J1")
 		(hatch edge 0.5)
 		(connect_pads
@@
 			(thermal_gap 0.5)
 			(thermal_bridge_width 0.5)
-			(island_removal_mode 1)
-			(island_area_min 10)
 		)
 		(polygon
 			(pts
-				(xy 41.5 32) (xy 41.5 38) (xy 43.5 38) (xy 43.5 32)
-			)
-		)
-	)
-	(zone
-		(net 0)
-		(net_name "")
-		(layer "F.Cu")
-		(hatch edge 0.5)
-		(connect_pads
-			(clearance 0.5)
-		)
-		(min_thickness 0.25)
-		(filled_areas_thickness no)
-		(fill
-			(thermal_gap 0.5)
-			(thermal_bridge_width 0.5)
-			(island_removal_mode 1)
-			(island_area_min 10)
-		)
-		(polygon
-			(pts
-				(xy 32 35.5) (xy 40.5 35.5) (xy 40.5 32) (xy 32 32)
-			)
-		)
-	)
-	(zone
-		(net 0)
-		(net_name "")
-		(layer "F.Cu")
-		(name "M1")
+				(xy 36.5 38.5) (xy 36.5 36.5) (xy 38.5 36.5) (xy 38.5 38.5)
+			)
+		)
+	)
+	(zone
+		(net 0)
+		(net_name "")
+		(layer "F.SilkS")
+		(name "transistor")
 		(hatch edge 0.5)
 		(connect_pads
@@
 			(thermal_gap 0.5)
 			(thermal_bridge_width 0.5)
+			(island_removal_mode 1)
+			(island_area_min 10)
 		)
 		(polygon
 			(pts
-				(xy 29 31.5) (xy 31 31.5) (xy 31 36) (xy 29 36)
-			)
-		)
-	)
-	(zone
-		(net 0)
-		(net_name "")
-		(layer "F.Cu")
+				(xy 32 32) (xy 40.5 32) (xy 40.5 35.5) (xy 32 35.5)
+			)
+		)
+	)
+	(zone
+		(net 0)
+		(net_name "")
+		(layer "F.SilkS")
+		(name "transistor")
+		(hatch edge 0.5)
+		(connect_pads
+			(clearance 0)
+		)
+		(min_thickness 0.25)
+		(filled_areas_thickness no)
+		(keepout
+			(tracks not_allowed)
+			(vias not_allowed)
+			(pads not_allowed)
+			(copperpour allowed)
+			(footprints allowed)
+		)
+		(placement
+			(enabled no)
+			(sheetname "")
+		)
+		(fill
+			(thermal_gap 0.5)
+			(thermal_bridge_width 0.5)
+			(island_removal_mode 1)
+			(island_area_min 10)
+		)
+		(polygon
+			(pts
+				(xy 41.5 32) (xy 41.5 38) (xy 43.5 38) (xy 43.5 32)
+			)
+		)
+	)
+	(zone
+		(net 0)
+		(net_name "")
+		(layer "F.SilkS")
 		(name "U2")
 		(hatch edge 0.5)
